Commit message: fixed package.xml with corrected upper plate dim

File: software/ros2_ws/src/tank_description/urdf/tank.urdf (robot description, URDF)
Before this commit: robot my_tank, 27 links, 26 joints
Links:
- link platform: geometry visual box size=0.257 0.152 0.002
Joints:
- joint lidar_standoff_fl_joint: origin xyz=0.042 0.032 0.015 -> xyz=0.034 0.032 0.015
- joint lidar_standoff_fr_joint: origin xyz=0.042 -0.032 0.015 -> xyz=0.034 -0.032 0.015
- joint lidar_standoff_rl_joint: origin xyz=-0.015 0.025 0.015 -> xyz=-0.023 0.025 0.015
- joint lidar_standoff_rr_joint: origin xyz=-0.015 -0.025 0.015 -> xyz=-0.023 -0.025 0.015

Commit message: new urdf

File: software/ros2_ws/src/tank_description/urdf/tank.urdf (robot description, URDF)
Before this commit: robot my_tank, 27 links, 26 joints
Links:
- removed link standoff_l4
- removed link standoff_r4
- removed link track_l_bottom
- removed link track_l_front
- removed link track_l_rear
- removed link track_l_top
- removed link track_r_bottom
- removed link track_r_front
- removed link track_r_rear
- removed link track_r_top
- added link imu_link
- added link ultrasonic_back_link; visual mesh filename=package://tank_description/meshes/ultrasonic_sensor.stl scale=0.001 0.001 0.001
- added link ultrasonic_front_link; visual mesh filename=package://tank_description/meshes/ultrasonic_sensor.stl scale=0.001 0.001 0.001
- added link ultrasonic_left_link; visual mesh filename=package://tank_description/meshes/ultrasonic_sensor.stl scale=0.001 0.001 0.001
- added link ultrasonic_right_link; visual mesh filename=package://tank_description/meshes/ultrasonic_sensor.stl scale=0.001 0.001 0.001
- link base_link: mass 0.5 -> 1.02; geometry collision box size=0.1833 0.1776 0.0423; visual mesh filename=package://tank_description/meshes/new_chassis.stl scale=0.001 0.001 0.001
- link left_bearing: geometry collision cylinder length=0.023 radius=0.019; visual cylinder length=0.023 radius=0.019
- link left_drive: geometry collision cylinder length=0.023 radius=0.019; visual cylinder length=0.023 radius=0.019
- link platform: geometry visual box size=0.2 0.152 0.002
- link right_bearing: geometry collision cylinder length=0.023 radius=0.019; visual cylinder length=0.023 radius=0.019
- link right_drive: geometry collision cylinder length=0.023 radius=0.019; visual cylinder length=0.023 radius=0.019
Joints:
- removed joint standoff_l4_joint
- removed joint standoff_r4_joint
- removed joint track_l_bottom_joint
- removed joint track_l_front_joint
- removed joint track_l_rear_joint
- removed joint track_l_top_joint
- removed joint track_r_bottom_joint
- removed joint track_r_front_joint
- removed joint track_r_rear_joint
- removed joint track_r_top_joint
- added joint imu_joint: type fixed, parent base_link, child imu_link, origin xyz=0.00 0 0.078 rpy=0 0 0
- added joint ultrasonic_back_joint: type fixed, parent base_link, child ultrasonic_back_link, origin xyz=-0.085 0.0 0.012 rpy=0 0 1.5708
- added joint ultrasonic_front_joint: type fixed, parent base_link, child ultrasonic_front_link, origin xyz=0.08 0.0 0.042 rpy=0 0 -1.5708
- added joint ultrasonic_left_joint: type fixed, parent base_link, child ultrasonic_left_link, origin xyz=0.01 0.05 0.042 rpy=0 0 0
- added joint ultrasonic_right_joint: type fixed, parent base_link, child ultrasonic_right_link, origin xyz=0.01 -0.05 0.042 rpy=0 0 3.1416
- joint left_bearing_joint: origin xyz=0.08 0.1 0 rpy=-1.5708 0 0 -> xyz=0.058 0.0686 0.001 rpy=-1.5708 0 0
- joint left_drive_joint: origin xyz=-0.0925 0.1 0 rpy=-1.5708 0 0 -> xyz=-0.0579 0.068 0.001 rpy=-1.5708 0 0
- joint lidar_joint: origin xyz=0 0 0.03 -> xyz=0.05 0 0.03
- joint lidar_standoff_fl_joint: origin xyz=0.034 0.032 0.015 -> xyz=0.072 0.032 0.015
- joint lidar_standoff_fr_joint: origin xyz=0.034 -0.032 0.015 -> xyz=0.072 -0.032 0.015
- joint lidar_standoff_rl_joint: origin xyz=-0.023 0.025 0.015 -> xyz=0.015 0.025 0.015
- joint lidar_standoff_rr_joint: origin xyz=-0.023 -0.025 0.015 -> xyz=0.015 -0.025 0.015
- joint platform_joint: origin xyz=0 0 0.09 -> xyz=0 0 0.082
- joint right_bearing_joint: origin xyz=-0.08 -0.1 0 rpy=-1.5708 0 0 -> xyz=-0.058 -0.069 0.001 rpy=-1.5708 0 0
- joint right_drive_joint: origin xyz=0.0925 -0.1 0 rpy=-1.5708 0 0 -> xyz=0.058 -0.068 0.001 rpy=-1.5708 0 0
- joint standoff_l1_joint: origin xyz=-0.125 0.068 0.063 -> xyz=0.015 0.044 0.057
- joint standoff_l2_joint: origin xyz=-0.0605 0.068 0.063 -> xyz=-0.067 0.044 0.057
- joint standoff_l3_joint: origin xyz=0.06 0.068 0.063 -> xyz=0.071 0.044 0.057
- joint standoff_r1_joint: origin xyz=-0.125 -0.068 0.063 -> xyz=0.015 -0.044 0.057
- joint standoff_r2_joint: origin xyz=-0.0605 -0.068 0.063 -> xyz=-0.067 -0.044 0.057
- joint standoff_r3_joint: origin xyz=0.06 -0.068 0.063 -> xyz=0.071 -0.044 0.057

Commit message: Add slam.launch.py for SLAM functionality and update tank.urdf mesh filename

File: software/ros2_ws/src/tank_description/urdf/tank.urdf (robot description, URDF)
Before this commit: robot my_tank, 22 links, 21 joints
Links:
- link lidar_link: geometry collision cylinder length=0.03 radius=0.035; visual mesh filename=package://tank_description/meshes/YDLIDAR_X3Pro.stl scale=0.001 0.001 0.001

Commit message: Fix LIDAR standoff positions and adjust base link orientation for correct alignment

File: software/ros2_ws/src/tank_description/urdf/tank.urdf (robot description, URDF)
Before this commit: robot my_tank, 22 links, 21 joints
Joints:
- joint lidar_joint: origin xyz=0.05 0 0.03 -> xyz=-0.05 0 0.03
- joint lidar_standoff_fl_joint: origin xyz=0.072 0.032 0.015 -> xyz=-0.072 0.032 0.015
- joint lidar_standoff_fr_joint: origin xyz=0.072 -0.032 0.015 -> xyz=-0.072 -0.032 0.015
- joint lidar_standoff_rl_joint: origin xyz=0.015 0.025 0.015 -> xyz=-0.015 0.025 0.015
- joint lidar_standoff_rr_joint: origin xyz=0.015 -0.025 0.015 -> xyz=-0.015 -0.025 0.015

Commit message: Fix LIDAR standoff positions and adjust base link orientation for correct alignment

File: software/ros2_ws/src/tank_description/urdf/tank.urdf (robot description, URDF)
Before this commit: robot my_tank, 22 links, 21 joints
Joints:
- joint lidar_joint: origin xyz=-0.05 0 0.03 -> xyz=0.05 0 0.03
- joint lidar_standoff_fl_joint: origin xyz=-0.072 0.032 0.015 -> xyz=0.072 0.032 0.015
- joint lidar_standoff_fr_joint: origin xyz=-0.072 -0.032 0.015 -> xyz=0.072 -0.032 0.015
- joint lidar_standoff_rl_joint: origin xyz=-0.015 0.025 0.015 -> xyz=0.015 0.025 0.015
- joint lidar_standoff_rr_joint: origin xyz=-0.015 -0.025 0.015 -> xyz=0.015 -0.025 0.015

Commit message: Fix odometry distance calculations and update URDF for correct base link and LIDAR orientations

File: software/ros2_ws/src/tank_description/urdf/tank.urdf (robot description, URDF)
Before this commit: robot my_tank, 22 links, 21 joints
Joints:
- joint lidar_joint: origin xyz=0.05 0 0.03 -> xyz=-0.05 0 0.03

Commit message: Fix IMU and LIDAR orientations in URDF for correct alignment

File: software/ros2_ws/src/tank_description/urdf/tank.urdf (robot description, URDF)
Before this commit: robot my_tank, 22 links, 21 joints
Joints:
- joint imu_joint: origin xyz=0.00 0 0.078 rpy=0 0 0 -> xyz=0.00 0 0.078 rpy=0 0 3.14159
- joint lidar_joint: origin xyz=-0.05 0 0.03 -> xyz=0.05 0 0.03

Commit message: Refine URDF link origins and orientations for improved accuracy

File: software/ros2_ws/src/tank_description/urdf/tank.urdf (robot description, URDF)
Before this commit: robot my_tank, 22 links, 21 joints
Joints:
- joint imu_joint: origin xyz=0.00 0 0.078 rpy=0 0 3.14159 -> xyz=0.000 0.000 0.078 rpy=0.000 0.000 3.14159
- joint left_bearing_joint: origin xyz=0.058 0.0686 0.001 rpy=-1.5708 0 0 -> xyz=0.058 0.0686 0.001 rpy=-1.5708 0.0 0.0
- joint left_drive_joint: origin xyz=-0.0579 0.068 0.001 rpy=-1.5708 0 0 -> xyz=-0.0579 0.068 0.001 rpy=-1.5708 0.0 0.0
- joint lidar_joint: origin xyz=0.05 0 0.03 -> xyz=0.050 0.000 0.030 rpy=0.000 0.000 3.14159
- joint lidar_standoff_fl_joint: origin xyz=0.072 0.032 0.015 -> xyz=0.072 0.032 0.015 rpy=0.0 0.0 0.0
- joint lidar_standoff_fr_joint: origin xyz=0.072 -0.032 0.015 -> xyz=0.072 -0.032 0.015 rpy=0.0 0.0 0.0
- joint lidar_standoff_rl_joint: origin xyz=0.015 0.025 0.015 -> xyz=0.015 0.025 0.015 rpy=0.0 0.0 0.0
- joint lidar_standoff_rr_joint: origin xyz=0.015 -0.025 0.015 -> xyz=0.015 -0.025 0.015 rpy=0.0 0.0 0.0
- joint platform_joint: origin xyz=0 0 0.082 -> xyz=0.0 0.0 0.082 rpy=0.0 0.0 0.0
- joint right_bearing_joint: origin xyz=-0.058 -0.069 0.001 rpy=-1.5708 0 0 -> xyz=-0.058 -0.069 0.001 rpy=-1.5708 0.0 0.0
- joint right_drive_joint: origin xyz=0.058 -0.068 0.001 rpy=-1.5708 0 0 -> xyz=0.058 -0.068 0.001 rpy=-1.5708 0.0 0.0
- joint standoff_l1_joint: origin xyz=0.015 0.044 0.057 -> xyz=0.015 0.044 0.057 rpy=0.0 0.0 0.0
- joint standoff_l2_joint: origin xyz=-0.067 0.044 0.057 -> xyz=-0.067 0.044 0.057 rpy=0.0 0.0 0.0
- joint standoff_l3_joint: origin xyz=0.071 0.044 0.057 -> xyz=0.071 0.044 0.057 rpy=0.0 0.0 0.0
- joint standoff_r1_joint: origin xyz=0.015 -0.044 0.057 -> xyz=0.015 -0.044 0.057 rpy=0.0 0.0 0.0
- joint standoff_r2_joint: origin xyz=-0.067 -0.044 0.057 -> xyz=-0.067 -0.044 0.057 rpy=0.0 0.0 0.0
- joint standoff_r3_joint: origin xyz=0.071 -0.044 0.057 -> xyz=0.071 -0.044 0.057 rpy=0.0 0.0 0.0
- joint ultrasonic_back_joint: origin xyz=-0.085 0.0 0.012 rpy=0 0 1.5708 -> xyz=-0.085 0.0 0.012 rpy=0.0 0.0 1.5708
- joint ultrasonic_front_joint: origin xyz=0.08 0.0 0.042 rpy=0 0 -1.5708 -> xyz=0.08 0.0 0.042 rpy=0.0 0.0 -1.5708
- joint ultrasonic_left_joint: origin xyz=0.01 0.05 0.042 rpy=0 0 0 -> xyz=0.01 0.05 0.042 rpy=0.0 0.0 0.0
- joint ultrasonic_right_joint: origin xyz=0.01 -0.05 0.042 rpy=0 0 3.1416 -> xyz=0.01 -0.05 0.042 rpy=0.0 0.0 3.14159

Commit message: Update nav2_params.yaml with explicit paths for behavior trees and fix plugin paths in tank.urdf for consistency

File: software/ros2_ws/src/tank_description/urdf/tank.urdf (robot description, URDF)
Before this commit: robot my_tank, 22 links, 21 joints
Links:
- link lidar_link: mass 0.05 -> None; geometry visual mesh filename=package://tank_description/meshes/ydlidar_x3pro.stl scale=0.001 0.001 0.001
Joints:
- joint imu_joint: origin xyz=0.000 0.000 0.078 rpy=0.000 0.000 3.14159 -> xyz=0.00 0 0.078 rpy=0 0 3.14159
- joint left_bearing_joint: origin xyz=0.058 0.0686 0.001 rpy=-1.5708 0.0 0.0 -> xyz=0.058 0.0686 0.001 rpy=-1.5708 0 0
- joint left_drive_joint: origin xyz=-0.0579 0.068 0.001 rpy=-1.5708 0.0 0.0 -> xyz=-0.0579 0.068 0.001 rpy=-1.5708 0 0
- joint lidar_joint: origin xyz=0.050 0.000 0.030 rpy=0.000 0.000 3.14159 -> xyz=0.05 0 0.03
- joint lidar_standoff_fl_joint: origin xyz=0.072 0.032 0.015 rpy=0.0 0.0 0.0 -> xyz=0.072 0.032 0.015
- joint lidar_standoff_fr_joint: origin xyz=0.072 -0.032 0.015 rpy=0.0 0.0 0.0 -> xyz=0.072 -0.032 0.015
- joint lidar_standoff_rl_joint: origin xyz=0.015 0.025 0.015 rpy=0.0 0.0 0.0 -> xyz=0.015 0.025 0.015
- joint lidar_standoff_rr_joint: origin xyz=0.015 -0.025 0.015 rpy=0.0 0.0 0.0 -> xyz=0.015 -0.025 0.015
- joint platform_joint: origin xyz=0.0 0.0 0.082 rpy=0.0 0.0 0.0 -> xyz=0 0 0.082
- joint right_bearing_joint: origin xyz=-0.058 -0.069 0.001 rpy=-1.5708 0.0 0.0 -> xyz=-0.058 -0.069 0.001 rpy=-1.5708 0 0
- joint right_drive_joint: origin xyz=0.058 -0.068 0.001 rpy=-1.5708 0.0 0.0 -> xyz=0.058 -0.068 0.001 rpy=-1.5708 0 0
- joint standoff_l1_joint: origin xyz=0.015 0.044 0.057 rpy=0.0 0.0 0.0 -> xyz=0.015 0.044 0.057
- joint standoff_l2_joint: origin xyz=-0.067 0.044 0.057 rpy=0.0 0.0 0.0 -> xyz=-0.067 0.044 0.057
- joint standoff_l3_joint: origin xyz=0.071 0.044 0.057 rpy=0.0 0.0 0.0 -> xyz=0.071 0.044 0.057
- joint standoff_r1_joint: origin xyz=0.015 -0.044 0.057 rpy=0.0 0.0 0.0 -> xyz=0.015 -0.044 0.057
- joint standoff_r2_joint: origin xyz=-0.067 -0.044 0.057 rpy=0.0 0.0 0.0 -> xyz=-0.067 -0.044 0.057
- joint standoff_r3_joint: origin xyz=0.071 -0.044 0.057 rpy=0.0 0.0 0.0 -> xyz=0.071 -0.044 0.057
- joint ultrasonic_back_joint: origin xyz=-0.085 0.0 0.012 rpy=0.0 0.0 1.5708 -> xyz=-0.085 0.0 0.012 rpy=0 0 1.5708
- joint ultrasonic_front_joint: origin xyz=0.08 0.0 0.042 rpy=0.0 0.0 -1.5708 -> xyz=0.08 0.0 0.042 rpy=0 0 -1.5708
- joint ultrasonic_left_joint: origin xyz=0.01 0.05 0.042 rpy=0.0 0.0 0.0 -> xyz=0.01 0.05 0.042 rpy=0 0 0
- joint ultrasonic_right_joint: origin xyz=0.01 -0.05 0.042 rpy=0.0 0.0 3.14159 -> xyz=0.01 -0.05 0.042 rpy=0 0 3.1416

Commit message: Normalize origin values in tank.urdf for consistency and clarity

File: software/ros2_ws/src/tank_description/urdf/tank.urdf (robot description, URDF)
Before this commit: robot my_tank, 22 links, 21 joints
Links:
- link lidar_link: geometry visual mesh filename=package://tank_description/meshes/YDLIDAR_X3Pro.stl scale=0.001 0.001 0.001
Joints:
- joint imu_joint: origin xyz=0.00 0 0.078 rpy=0 0 3.14159 -> xyz=0.000 0.000 0.078 rpy=0.000 0.000 3.14159
- joint left_bearing_joint: origin xyz=0.058 0.0686 0.001 rpy=-1.5708 0 0 -> xyz=0.058 0.0686 0.001 rpy=-1.5708 0.000 0.000
- joint left_drive_joint: origin xyz=-0.0579 0.068 0.001 rpy=-1.5708 0 0 -> xyz=-0.0579 0.068 0.001 rpy=-1.5708 0.000 0.000
- joint lidar_joint: origin xyz=0.05 0 0.03 -> xyz=0.050 0.000 0.030
- joint platform_joint: origin xyz=0 0 0.082 -> xyz=0.000 0.000 0.082
- joint right_bearing_joint: origin xyz=-0.058 -0.069 0.001 rpy=-1.5708 0 0 -> xyz=-0.058 -0.069 0.001 rpy=-1.5708 0.000 0.000
- joint right_drive_joint: origin xyz=0.058 -0.068 0.001 rpy=-1.5708 0 0 -> xyz=0.058 -0.068 0.001 rpy=-1.5708 0.000 0.000
- joint ultrasonic_back_joint: origin xyz=-0.085 0.0 0.012 rpy=0 0 1.5708 -> xyz=-0.085 0.000 0.012 rpy=0.000 0.000 1.5708
- joint ultrasonic_front_joint: origin xyz=0.08 0.0 0.042 rpy=0 0 -1.5708 -> xyz=0.08 0.000 0.042 rpy=0.000 0.000 -1.5708
- joint ultrasonic_left_joint: origin xyz=0.01 0.05 0.042 rpy=0 0 0 -> xyz=0.01 0.05 0.042 rpy=0.000 0.000 0.000
- joint ultrasonic_right_joint: origin xyz=0.01 -0.05 0.042 rpy=0 0 3.1416 -> xyz=0.01 -0.05 0.042 rpy=0.000 0.000 3.1416

Commit message: Refine odometry handling and update EKF and SLAM configurations for improved accuracy and performance

File: software/ros2_ws/src/tank_description/urdf/tank.urdf (robot description, URDF)
Before this commit: robot my_tank, 22 links, 21 joints
Joints:
- joint imu_joint: origin xyz=0.000 0.000 0.078 rpy=0.000 0.000 3.14159 -> xyz=0.000 0.000 0.078 rpy=0.000 0.000 0.000

Commit message: Fix LIDAR orientation in tank.urdf for accurate positioning

File: software/ros2_ws/src/tank_description/urdf/tank.urdf (robot description, URDF)
Before this commit: robot my_tank, 22 links, 21 joints
Joints:
- joint lidar_joint: origin xyz=0.050 0.000 0.030 -> xyz=0.050 0.000 0.030 rpy=0.000 0.000 3.1416
